File: hardware/femtobuck.sch (EAGLE design)
At the start: 16 parts, among them U1 AL8805

Commit message: AL8805 Buck LED driver EOL, replace with AL8860
Parts:
- CH1: device SparkFun:M023.5MM_LOCK -> SparkFun-Connectors:CONN_023.5MM_LOCK
- L1: value 33uH -> 33µH/±20%/1.4A; device SparkFun-Passives:INDUCTORBOURNS_SRN6045 -> SparkFun-Coils:INDUCTOR-SRN6045-33UH
- SJ2: device SparkFun-Passives:JUMPER-PAD-2-NO -> SparkFun-Jumpers:JUMPER-SMT_2_NO_NO-SILK
- U1: value AL8805 -> AL8860; device SparkFun-PowerIC:AL8805 -> SparkFun-IC-Special-Function:AL8860
Other:
- note added: "Revised by: Priyanka Makin"
- note added: "v13"
- note removed: "12"
